File: projects/telemetry/telemetry_core/telemetry_core.kicad_pcb (KiCad board)
At the start: 2 copper layers, 109.3 x 58.3 mm, 19 parts, among them U101 TPS560430YF

Commit message: fix MCP79511, start layout
Parts:
- added C1: C_0.1uF, footprints:C_0805_OEM, F.Cu at (52.8, 100.1)
- added C10: C_10pf, footprints:C_10pf, F.Cu at (105.9, 240.5)
- added C11: C_0.1uF, footprints:C_0805_OEM, F.Cu at (123.1, 210.8)
- added C12: C_10nF, footprints:C_1206_OEM, F.Cu at (128.9, 238.4)
- added C13: C_0.1uF, footprints:C_0805_OEM, F.Cu at (40.4, 65.9)
- added C14: C_0.1uF, footprints:C_0805_OEM, F.Cu at (48.4, 64.9)
- added C15: C_radial_10mm_5mm, footprints:C_radial_10mm_5mm, F.Cu at (50.2, 169.4)
- added C16: C_0.1uF, footprints:C_0805_OEM, F.Cu at (48.6, 89.7)
- added C2: C_100pF, footprints:C_0805_OEM, F.Cu at (58.5, 84.4)
- added C5: C_30pF, footprints:C_0805_OEM, F.Cu at (55.2, 119.6)
- added C7: C_30pF, footprints:C_0805_OEM, F.Cu at (75.1, 215.1)
- added C8: C_0.1uF, footprints:C_0805_OEM, F.Cu at (106.3, 209.8)
- added C9: C_10pf, footprints:C_10pf, F.Cu at (105.5, 245.0)
- added D4: LED_0805, footprints:LED_0805_OEM, F.Cu at (11.0, 241.2)
- added D5: LED_0805, footprints:LED_0805_OEM, F.Cu at (7.87, 241.2)
- added D6: LED_0805, footprints:LED_0805_OEM, F.Cu at (4.70, 241.3)
- added D7: BAT400D-7-F, footprints:SOT-23-3_OEM, F.Cu at (42.9, 168.5)
- added J1: MM_F_RA_20, footprints:micromatch_female_ra_20, F.Cu at (29.1, 170.9)
- added J2: JST_SM06B-GHS-TB_LF__SN_, footprints:JST_SM06B-GHS-TB_LF__SN_, F.Cu at (204.6, 128.3)
- added J3: CONN_02X03, footprints:Pin_Header_Straight_2x03, F.Cu at (201.4, 80.4)
- added L1: L_100uH, footprints:L_100uH_OEM, F.Cu at (77.5, 240.6)
- added R1: R_100, footprints:R_0805_OEM, F.Cu at (74.8, 220.9)
- added R11: R_475, footprints:R_0805_OEM, F.Cu at (133.0, 249.2)
- added R12: R_120_DNP, footprints:R_0805_OEM, F.Cu at (80.4, 213.9)
- added R5: R_10K, footprints:R_0805_OEM, F.Cu at (53.6, 223.3)
- added R7: R_200, footprints:R_0805_OEM, F.Cu at (11.3, 236.2)
- added R8: R_200, footprints:R_0805_OEM, F.Cu at (8.26, 235.7)
- added R9: R_200, footprints:R_0805_OEM, F.Cu at (5.08, 236.2)
- added TP1: Test_Point_SMD, footprints:Test_Point_SMD, F.Cu at (15.5, 230.8)
- added TP2: Test_Point_SMD, footprints:Test_Point_SMD, F.Cu at (7.11, 222.8)
- added TP3: Test_Point_SMD, footprints:Test_Point_SMD, F.Cu at (-1.65, 230.6)
- added TP4: Test_Point_SMD, footprints:Test_Point_SMD, F.Cu at (54.2, 234.2)
- added TP5: Test_Point_SMD, footprints:Test_Point_SMD, F.Cu at (46.4, 233.8)
- added TP6: Test_Point_SMD, footprints:Test_Point_SMD, F.Cu at (34.7, 234.9)
- added U1: ATMEGA16M1, footprints:TQFP-32_7x7mm_Pitch0.8mm, F.Cu at (52.3, 109.7)
- added U3: MCP79511-I_MS, footprints:MCP79511_I_MS, F.Cu at (120.8, 244.7)
- added U4: TXB0104PW, Package_SO:TSSOP-14_4.4x5mm_P0.65mm, F.Cu at (113.5, 209.9)
- added U5: LM3480-3.3, Package_TO_SOT_SMD:SOT-23, F.Cu at (47.4, 71.8)
- added U6: MCP2561-E_SN, footprints:SOIC-8_3.9x4.9mm_Pitch1.27mm_OEM, F.Cu at (30.7, 107.2)
- added Y1: Crystal_SMD, footprints:Crystal_SMD_FA238, F.Cu at (76.0, 211.8)
- added Y2: Crystal_32_768kHz, footprints:Crystal_32_768kHZ, F.Cu at (108.7, 251.6)
- renumbered C101 to C3, C102 to C4, C103 to C6, COUT101 to COUT1, COUT102 to COUT2, COUT103 to COUT3, D101 to D1, D102 to D2, D103 to D3, F101 to F1, R104 to R10, R101 to R2, R102 to R3, R103 to R4, R105 to R6, U101 to U2
Connections:
- C6 pad 2: Net-(C103-Pad2) -> Net-(C6-Pad2)
- COUT1 pad 1: Net-(COUT101-Pad1) -> Net-(COUT1-Pad1)
- COUT2 pad 1: Net-(COUT101-Pad1) -> Net-(COUT1-Pad1)
- COUT3 pad 1: Net-(COUT101-Pad1) -> Net-(COUT1-Pad1)
- R10 pad 1: Net-(COUT101-Pad1) -> +5V
- R10 pad 2: VCC -> Net-(COUT1-Pad1)
- R4 pad 1: Net-(COUT101-Pad1) -> Net-(COUT1-Pad1)
- R6 pad 1: VCC -> Net-(COUT1-Pad1)
- U2 pad 6: Net-(C103-Pad2) -> Net-(C6-Pad2)
Routing:
- net VCC: track 22.7 -> 0.00 mm
- net Net-(COUT1-Pad1): track 0.00 -> 22.7 mm
