File: projects/telemetry/go_kart_telemetry_core/go_kart_telemetry_core.kicad_pcb (KiCad board)
At the start: 2 copper layers, 76.2 x 63.5 mm, 59 parts, among them J1 MM_F_RA_20, J2 JST_SM06B-GHS-TB_LF__SN_, J3 CONN_02X03, U1 ATMEGA16M1, U2 TPS560430YF, U3 MCP79511-I_MS, U4 TXB0104PW, U5 LM3480-3.3, U6 MCP2561-E_SN, Y1 Crystal_SMD, Y2 Crystal_32_768kHz

Commit message: feat: begin changes for gokart
Parts:
- removed C6: C_0.1uF, footprints:C_0805_OEM
- removed COUT1: C_22uF, footprints:C_1206_OEM
- removed COUT2: C_33uF, footprints:Fuse_1812
- removed COUT3: C_47uF, footprints:C_0805_OEM
- removed L101: L_100uH, footprints:L_100uH_OEM
- removed R3: R_25K, footprints:R_0805_OEM
- removed R4: R_100K, footprints:R_0805_OEM
- added J4: MM_F_RA_04, footprints:micromatch_female_ra_4, F.Cu at (88.2, 119.9)
- C3: value C_0.1uF -> C_1uF
- C4: value C_2.2uF -> C_1uF; footprint footprints:C_0603_1608Metric -> footprints:C_0805_OEM
- J1: value MM_F_RA_20 -> MM_F_RA_04; footprint footprints:micromatch_female_ra_20 -> footprints:micromatch_female_ra_4
- U2: value TPS560430YF -> AP7370; footprint footprints:SOT-23-6_OEM -> footprints:SOT-23-5
- moved D2 95.5 mm to (85.4, 104.5), turned to 0 degrees
- moved D1 90.4 mm to (86.8, 100.6)
- moved TP6 87.7 mm to (99.9, 95.4), turned to 0 degrees
- moved R10 86.5 mm to (87.3, 95.7), turned to 0 degrees
- moved C3 83.9 mm to (94.9, 117.3)
- moved C4 83.7 mm to (94.9, 120.1)
- moved U2 83.6 mm to (95.1, 113.6), turned to 0 degrees
- moved F1 81.2 mm to (93.3, 104.2), turned to 0 degrees
- moved TP5 79.3 mm to (93.3, 100.1), turned to 0 degrees
- moved R2 79.0 mm to (98.2, 101.5)
- moved TP4 76.5 mm to (94.4, 95.4), turned to 0 degrees
- moved D3 67.2 mm to (98.6, 98.7)
- moved R6 66.5 mm to (103.1, 98.8), turned to 0 degrees
- moved J1 59.5 mm to (104.6, 114.2), turned to 180 degrees
Connections:
- C4 pad 1: Net-(C3-Pad1) -> Net-(C4-Pad1)
- R10 pad 2: Net-(COUT1-Pad1) -> Net-(C4-Pad1)
- R6 pad 1: Net-(COUT1-Pad1) -> Net-(C4-Pad1)
- U2 pad 1: Net-(C6-Pad1) -> Net-(C3-Pad1)
- U2 pad 3: Net-(R3-Pad1) -> (no net)
- U2 pad 4: Net-(C3-Pad1) -> (no net)
- U2 pad 5: Net-(C3-Pad1) -> Net-(C4-Pad1)
Routing:
- net GND: track 100.6 -> 48.2 mm, vias 36 -> 23
- net Net-(C3-Pad1): track 22.9 -> 0.00 mm
- net Net-(COUT1-Pad1): track 21.7 -> 0.00 mm
- net /MISO: track 46.5 -> 29.8 mm
- net /CAN_P: track 36.6 -> 21.2 mm
- net +5V: track 143.6 -> 130.3 mm
- net /CAN_N: track 31.1 -> 18.0 mm
- net /12V: track 27.2 -> 16.1 mm
- net Net-(C6-Pad2): track 5.44 -> 0.00 mm
- net /12V_IN: track 4.25 -> 0.00 mm
- net Net-(R3-Pad1): track 4.18 -> 0.00 mm
- net Net-(C6-Pad1): track 2.39 -> 0.00 mm
- net Net-(D3-Pad2): track 1.75 -> 0.00 mm
- net Net-(D2-Pad2): track 1.75 -> 0.00 mm
- removed copper zone on F.Cu, net GND
- removed copper zone on F.Cu, net Net-(C6-Pad1)
- removed copper zone on F.Cu, net Net-(C6-Pad2)
- removed copper zone on F.Cu, net Net-(COUT1-Pad1)
Other:
- board text removed: "12V"
- board text removed: "5V"
- board text removed: "GND"
