File: projects/hitl/hardware/primary_board/connectors.kicad_sch (KiCad schematic)
At the start: 24 parts, among them J13 CONN_01x02, J14 SSW-122-01-G-D, J15 CONN_01x02, J2 Barrel_jack, J21 Screw_Terminal_01x03, J3 MM_F_VT_08_SM, J4 MM_F_VT_08_SM, J6 CONN_01x02

Commit message: Switch FTPROG to button and update I2C level shifter
Parts:
- J21: DigikeyLink (none) -> https://www.digikey.com/en/products/detail/phoenix-contact/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; DigikeyPartNumber (none) -> 277-1578-ND; MPN (none) -> 1935174
Changed lines of the file:
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@@
       (effects (font (size 1.27 1.27)) hide)
     )
-    (property "Datasheet" "~" (id 3) (at 214.376 34.29 0)
+    (property "Datasheet" "https://media.digikey.com/pdf/Data%20Sheets/Phoenix%20Contact%20PDFs/1935174.pdf" (id 3) (at 214.376 34.29 0)
       (effects (font (size 1.27 1.27)) hide)
     )
+    (property "DigikeyLink" "https://www.digikey.com/en/products/detail/phoenix-contact/1935174/568615" (id 4) (at 214.376 34.29 0)
+      (effects (font (size 1.27 1.27)) hide)
+    )
+    (property "MPN" "1935174" (id 5) (at 214.376 34.29 0)
+      (effects (font (size 1.27 1.27)) hide)
+    )
+    (property "DigikeyPartNumber" "277-1578-ND" (id 6) (at 214.376 34.29 0)
+      (effects (font (size 1.27 1.27)) hide)
+    )
