File: projects/hitl/hardware/primary_board/hitl-primary.kicad_sch (KiCad schematic)
At the start: 90 parts, among them J1 USB-Micro-1981568-1, J10 CONN_01X03, J11 CONN_01X03, J12 CONN_01X03, J13 CONN_01x02, J14 SSW-122-01-G-D, J15 CONN_01x02, J2 Barrel_jack, J3 MM_F_VT_08_SM, J4 MM_F_VT_08_SM, J5 CONN_01x02, J6 DSub-9, J7 CONN_01X03, J8 CONN_01X03, J9 CONN_01X03, Q1 SSM3K333R, Q2 SSM3K333R, Q3 SSM3K333R, Q4 SSM3K333R, U1 R_500, U2 FT4222H, U3 PCA9306, U4 AD5675, U5 MAX7300AAXT, Y1 Crystal_12MHz

Commit message: Split schematic into sheets
Parts:
- removed C1, C10, C13, C15, C8: C_4.7uF_25V, footprints:C_0805_OEM, symbol formula:C_4.7uF_25V
- removed C11, C14, C2, C9: C_100nF, footprints:C_0603_1608Metric, symbol formula:C_100nF
- removed C12, C29, C4, C5, C6: C_10uF_50V, footprints:C_0805_OEM, symbol formula:C_10uF_50V
- removed C16: C_100pF, footprints:C_0805_OEM, symbol formula:C_100pF
- removed C17: C_10uF_16V, footprints:C_0805_OEM, symbol formula:C_10uF_16V
- removed C18: C_0.1uF, footprints:C_0805_OEM, symbol formula:C_0.1uF
- removed C19: C_10uF_25V, footprints:C_0805_OEM, symbol formula:C_10uF_25V
- removed C3, C7: C_30pF, footprints:C_0805_OEM, symbol formula:C_30pF
- removed D1, D3: LED_0805, footprints:LED_0805_OEM, symbol formula:LED_0805
- removed D2: D_Zener_13V, footprints:D_13V_Zener, symbol formula:D_Zener_13V
- removed D4: LED_0805_Red, footprints:LED_0805_OEM, symbol formula:LED_0805_Red
- removed D5, D6: LED_0805_Amber, footprints:LED_0805_OEM, symbol formula:LED_0805_Amber
- removed F1: F_500mA_16V, footprints:Fuse_1210, symbol formula:F_500mA_16V
- removed F2: 1.5A_Fuse, footprints:Fuse_1206, symbol formula:1.5A_Fuse
- removed J1: USB-Micro-1981568-1, footprints:TE_1981568-1, symbol formula:USB-Micro-1981568-1
- removed J10, J11, J12, J7, J8, J9: CONN_01X03, footprints:PinHeader_1x03_P2.54mm_Vertical, symbol formula:CONN_01X03
- removed J13, J15, J5: CONN_01x02, footprints:pinheader_1x2, symbol formula:CONN_01x02
- removed J14: SSW-122-01-G-D, footprints:SAMTEC_SSW-122-01-G-D, symbol formula:SSW-122-01-G-D
- removed J2: Barrel_jack, footprints:barrel_jack_PJ-037A, symbol formula:Barrel_jack
- removed J3, J4: MM_F_VT_08_SM, footprints:micromatch_female_vert_8_sm, symbol formula:MM_F_VT_08_SM
- removed J6: DSub-9, footprints:TE_5745781-4, symbol formula:DSub-9
- removed Q1, Q2, Q3, Q4: SSM3K333R, footprints:SOT-23F, symbol formula:SSM3K333R
- removed R1, R6, R8: R_12K, footprints:R_0805_OEM, symbol formula:R_12K
- removed R10, R11, R44, R45: R_0, footprints:R_0603_1608Metric, symbol formula:R_0
- removed R12, R14, R21, R22: R_8.06k, footprints:R_0805_OEM, symbol formula:R_8.06k
- removed R13, R15, R17, R24, R26, R3, R5: R_10K, footprints:R_0805_OEM, symbol formula:R_10K
- removed R16: R_120_DNP, footprints:R_0805_OEM, symbol formula:R_120_DNP
- removed R18, R25, R27, R7: R_1.91K, footprints:R_0805_OEM, symbol formula:R_1.91K
- removed R19: R_200K, footprints:R_0805_OEM, symbol formula:R_200K
- removed R2, R9: R_3.01K, footprints:R_0805_OEM, symbol formula:R_3.01K
- removed R20: R_39K, footprints:R_0805_OEM, symbol formula:R_39K
- removed R4: R_1M, footprints:R_0805_OEM, symbol formula:R_1M
- removed TP1, TP2, TP3, TP4, TP5, TP6, TP7, TP8: Test_Point_SMD, footprints:Test_Point_SMD, symbol formula:Test_Point_SMD
- removed U1: R_500, footprints:R_0805_OEM, symbol formula:R_500
- removed U2: FT4222H, footprints:FT4222_QFN, symbol formula:FT4222H
- removed U3: PCA9306, footprints:SOP50P310X90-8N_pca9306, symbol formula:PCA9306
- removed U4: AD5675, footprints:SOP65P640X120-20N_AD, symbol formula:AD5675
- removed U5: MAX7300AAXT, footprints:SOP80P1030X264-36N, symbol formula:MAX7300AAXT
- removed Y1: Crystal_12MHz, footprints:Crystal_SMD_FA238, symbol formula:Crystal_12MHz
Connections:
- net ADC4 renamed ADC Circuitry/ADC_SELF_TEST
- net VOUT-8 renamed DAC8
- no-connect marks 16 -> 3
Other:
- added sheet Connectors (connectors.kicad_sch)
- added sheet DAC (dac.kicad_sch)
- added sheet GPIO (gpio.kicad_sch)
- added sheet USB->I2C (usb.kicad_sch)
- sheet ADC Circuitry ports: added ADC[1..7], ADC_MUX0, ADC_MUX1, ADC_MUX2, ADC_SELF_TEST, USB_5V; removed ADC-1, ADC-2, ADC-4, AMUX-1, AMUX-2, AMUX-3, AMUX-4, AMUX-5, AMUX-6, AMUX-7, CA0, CA1, GPIO-18, GPIO-19, GPIO-20, GPIO-21
- sheet VBus Power ports: added SCL, SCL-FT, SDA, SDA-FT; removed none
- note added: "ADC/DAC Introspection Testing"
- note added: "GPIO Signals for Analog Mux"
- note added: "SCL"
- note added: "SDA"
- note added: "Signal used to change all DAC pins at once"
- note added: "Signal used to sense USB Vbus voltage"
- note removed: "12V Barrel Jack"
- note removed: "5V (output)"
- note removed: "Address Start: 030......"
- note removed: "Analog -> Digital"
- note removed: "Away From Primary"
- note removed: "CAN USB Adapter"
- note removed: "Device Under Test Connector"
- note removed: "Digital -> Analog"
- note removed: "FT Programming"
- note removed: "Gain = 1"
- note removed: "General Purpose Input/Output"
- note removed: "I2C Level Shifter"
- note removed: "Introspection Testing"
- note removed: "Operating in Mode 0 See pg.13 for more info"
- note removed: "Programming LEDs"
- note removed: "Secondary Board Connectors"
- note removed: "Should we add more address options? There are currently 4 which would cover the entire vehicle"
- note removed: "Sink 10mA Source 4.5mA"
- note removed: "Towards Primary"
- note removed: "USB Communication"
- note removed: "Vout = Vin * ~0.2 Vout ≈ 1V"
- note removed: "Vout = Vin * ~0.2 Vout ≈ 2.4V"
- note removed: "Vout0 thru Vout3 can Source/Sink 40mA Vout4 thru Vout7 can Source/Sink 40mA"
- note removed: "Will interface with: IPEH-002021 P-CAN USB"
- note removed: "https://www.digikey.com/en/products/detail/samtec-inc/SSW-122-01-G-D/1112036"
- note removed: "https://www.digikey.com/en/products/detail/w%C3%BCrth-elektronik/61304421121/4846887"
- note removed: "~5mA"
